File: boards/td4-shield-rev.1/td4-shield.kicad_pcb (KiCad board)
At the start: 2 copper layers, 57.2 x 53.3 mm, 86 parts, among them P1 Power, P2 Analog, P3 Digital, P4 Digital, P5 CONN_01X01, P6 CONN_01X01, P7 CONN_01X01, P8 CONN_01X01, SW1 INPUT, SW18 Manual Clock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

Commit message: Update kicad_pcb and gerber
Silk modified.
Parts:
- added LOGO1: OSHW-Logo2_9.8x8mm_SilkScreen, Symbols:OSHW-Logo2_9.8x8mm_SilkScreen, B.Cu at (173.0, 82.7)
