File: boards/td4-shield-rev.1/td4-shield.kicad_pcb (KiCad board)
At the start: 2 copper layers, 57.2 x 53.3 mm, 87 parts, among them P1 Power, P2 Analog, P3 Digital, P4 Digital, P5 CONN_01X01, P6 CONN_01X01, P7 CONN_01X01, P8 CONN_01X01, SW1 INPUT, SW18 Manual Clock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

Commit message: Fix the bugs on wiring to U2, U3, U4, and U5.
Connections:
- U2 pad 1: /3(**) -> /2
- U2 pad 2: /2 -> /3(**)
- U3 pad 1: /3(**) -> /2
- U3 pad 2: /2 -> /3(**)
- U4 pad 1: /3(**) -> /2
- U4 pad 2: /2 -> /3(**)
- U5 pad 1: /3(**) -> /2
- U5 pad 2: /2 -> /3(**)
Routing:
- net /IN3: track 90.4 -> 49.3 mm, vias 2 -> 0
- net GND: track 404.4 -> 383.2 mm, vias 1 -> 5
- net ROM_A0: track 12.2 -> 31.6 mm, vias 1 -> 0
- net /3(**): track 171.6 -> 153.2 mm, vias 2 -> 1
- net /ALU_S3: track 104.6 -> 121.8 mm, vias 2 -> 4
- net /IN1: track 81.4 -> 65.5 mm, vias 2 -> 0
- net ROM_D5: track 63.9 -> 48.2 mm
- net Net-(C4-Pad1): track 31.6 -> 16.1 mm
- net /ALU_S4: track 100.9 -> 116.4 mm
- net VCC: track 267.7 -> 257.6 mm, vias 7 -> 9
- net /RB1: track 23.7 -> 13.7 mm
- net /IN4: track 47.7 -> 37.8 mm
- net /~FLG_C: track 36.2 -> 26.9 mm, vias 0 -> 2
- net ROM_D2: track 36.0 -> 27.6 mm
- net Net-(R10-Pad2): track 41.9 -> 34.0 mm
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Other:
- board text added: "+3V3"
- board text added: "+5V"
- board text added: "ROM_A0"
- board text added: "ROM_A1"
- board text added: "ROM_A2"
- board text added: "ROM_A3"
- board text added: "ROM_D0"
- board text added: "ROM_D1"
- board text added: "ROM_D2"
- board text added: "ROM_D3"
- board text added: "ROM_D4"
- board text added: "ROM_D5"
- board text added: "ROM_D6"
- board text added: "ROM_D7"
